Commit message: robot model updated

File: robot_model/mmo_700/mmo_700.urdf.xacro (robot description, xacro)
@@ -10,5 +10,11 @@
   <xacro:include filename="$(find neo_mmo_700)/robot_model/mmo_700/urdf/xacros/mpo_700_body.xacro" />
   <!-- SENSORS -->
-  <xacro:include filename="$(find neo_mmo_700)/robot_model/mmo_700/urdf/xacros/sick_laser.xacro" />
+  <!-- Sick S300 - Comment/Uncomment if required  -->
+  <xacro:include filename="$(find neo_mmo_700)/robot_model/mmo_700/urdf/xacros/sick_S300.xacro" />
+  <!-- Microscan - Comment/Uncomment if required -->
+  <!-- <xacro:include filename="$(find neo_mmo_700)/robot_model/mmo_700/urdf/xacros/micro_scan.xacro" /> -->
+  <!-- USS and IMU - Comment/Uncomment if required  -->
+  <!-- <xacro:include filename="$(find neo_mmo_700)/robot_model/mmo_700/urdf/xacros/imu.xacro" />
+    <xacro:include filename="$(find neo_mmo_700)/robot_model/mmo_700/urdf/xacros/ultrasonic.xacro" /> -->
   <!-- Gazebo -->
   <xacro:include filename="$(find neo_mmo_700)/robot_model/mmo_700/urdf/xacros/mpo_700_gazebo.xacro" />
@@ -45,18 +51,17 @@
   </xacro:mmo_700_wheel>
 <!-- Sensors -->
-  <xacro:sick_v0 name="sick_laser_front" parent="base_link" ros_topic="laser_1/scan">
+  <xacro:sick_laser_v0 name="lidar_1" parent="base_link" ros_topic="lidar_1/scan_filtered">
     <origin xyz="0.360 0 0.181" rpy="3.14 0 0 " />
-  </xacro:sick_v0>
-  <xacro:sick_v0 name="sick_laser_back" parent="base_link" ros_topic="laser_2/scan">
+  </xacro:sick_laser_v0>
+  <xacro:sick_laser_v0 name="lidar_2" parent="base_link" ros_topic="lidar_2/scan_filtered">
     <origin xyz="-0.360 0 0.181" rpy="3.14 0 3.14" />
-  </xacro:sick_v0>
- <!--+++++++++++++++++++ IMU ++++++++++++++++++++++++-->
-  <!-- SENSORS -->
-  <xacro:include filename="$(find neo_mmo_700)/robot_model/mmo_700/urdf/xacros/imu.xacro" />
-  <xacro:imu name="imu_1" parent="base_link">
+  </xacro:sick_laser_v0>
+     <!--+++++++++++++++++++ IMU ++++++++++++++++++++++++-->
+ <!-- Comment or uncomment based on your requirement -->
+<!--   <xacro:imu name="imu_1" parent="base_link">
     <origin xyz="0.100 0 0.300" rpy="0 0 3.14" />
-  </xacro:imu>
+  </xacro:imu> -->
   <!--+++++++++++++++++++ Ultra Sonic ++++++++++++++++++++++++-->
-  <xacro:include filename="$(find neo_mmo_700)/robot_model/mmo_700/urdf/xacros/ultrasonic.xacro" />
+  <!-- Comment or uncomment based on your requirement -->
   <!-- SENSOR 1 -->
   <!-- xacro:us_sensor name="us_1" parent="base_link">

File: robot_model/mmo_700/urdf/xacros/imu.xacro (robot description, xacro)
@@ -1,4 +1,4 @@
 <?xml version="1.0"?>
-<robot xmlns:xacro="http://www.ros.org/wiki/xacro" name="mp_400">
+<robot xmlns:xacro="http://www.ros.org/wiki/xacro" name="mmo_700">
   <xacro:macro name="imu" params="name parent *origin">
     <joint name="${name}_joint" type="fixed">

File: robot_model/mmo_700/urdf/xacros/mpo_700_body.xacro (robot description, xacro)
@@ -1,4 +1,4 @@
 <?xml version="1.0"?>
-<robot xmlns:xacro="http://www.ros.org/wiki/xacro" name="mpo_700">
+<robot xmlns:xacro="http://www.ros.org/wiki/xacro" name="mmo_700">
   <xacro:macro name="mpo_700_base" params="name">
     <link name="${name}">

File: robot_model/mmo_700/urdf/xacros/mpo_700_gazebo.xacro (robot description, xacro)
@@ -5,6 +5,6 @@
     <self_collide>false</self_collide>
   </gazebo>
-  <gazebo reference="sick_laser_front_link">
-      <sensor type="ray" name="sick_laser_front_sensor">
+  <gazebo reference="lidar_1_link">
+      <sensor type="ray" name="lidar_1_sensor">
           <pose>0 0 0 0 0 0</pose>
           <visualize>false</visualize>
@@ -34,12 +34,12 @@
             </noise>
           </ray>
-          <plugin name="sick_laser_front" filename="libgazebo_ros_laser.so">
-            <topicName>laser_1/scan</topicName>
-            <frameName>sick_laser_front_link</frameName>
+          <plugin name="lidar_1" filename="libgazebo_ros_laser.so">
+            <topicName>lidar_1/scan_filtered</topicName>
+            <frameName>lidar_1_link</frameName>
           </plugin>
         </sensor>
   </gazebo>
-  <gazebo reference="sick_laser_back_link">
-      <sensor type="ray" name="sick_laser_back_sensor">
+  <gazebo reference="lidar_2_link">
+      <sensor type="ray" name="lidar_2_sensor">
           <pose>0 0 0 0 0 0</pose>
           <visualize>false</visualize>
@@ -69,11 +69,70 @@
             </noise>
           </ray>
-          <plugin name="sick_laser_back" filename="libgazebo_ros_laser.so">
-            <topicName>laser_2/scan</topicName>
-            <frameName>sick_laser_back_link</frameName>
+          <plugin name="lidar_2" filename="libgazebo_ros_laser.so">
+            <topicName>lidar_2/scan_filtered</topicName>
+            <frameName>lidar_2_link</frameName>
           </plugin>
         </sensor>
   </gazebo>
-  <gazebo>
+    <gazebo reference="imu_link">
+    <gravity>true</gravity>
+    <sensor name="imu_sensor" type="imu">
+      <always_on>true</always_on>
+      <update_rate>100</update_rate>
+      <visualize>true</visualize>
+      <topic>__default_topic__</topic>
+      <plugin filename="libgazebo_ros_imu_sensor.so" name="imu_plugin">
+        <topicName>imu</topicName>
+        <bodyName>imu_link</bodyName>
+        <updateRateHZ>10.0</updateRateHZ>
+        <gaussianNoise>0.0</gaussianNoise>
+        <xyzOffset>0 0 0</xyzOffset>
+        <rpyOffset>0 0 0</rpyOffset>
+        <frameName>imu_link</frameName>
+      </plugin>
+      <pose>0 0 0 0 0 0</pose>
+    </sensor>
+  </gazebo>
+    <!-- camera -->
+  <gazebo reference="camera_link">
+    <sensor type="camera" name="camera1">
+      <update_rate>30.0</update_rate>
+      <camera name="head">
+        <horizontal_fov>1.3962634</horizontal_fov>
+        <image>
+          <width>800</width>
+          <height>800</height>
+          <format>R8G8B8</format>
+        </image>
+        <clip>
+          <near>0.02</near>
+          <far>300</far>
+        </clip>
+        <noise>
+          <type>gaussian</type>
+          <!-- Noise is sampled independently per pixel on each frame.
+               That pixel's noise value is added to each of its color
+               channels, which at that point lie in the range [0,1]. -->
+          <mean>0.0</mean>
+          <stddev>0.007</stddev>
+        </noise>
+      </camera>
+      <plugin name="camera_controller" filename="libgazebo_ros_camera.so">
+        <alwaysOn>true</alwaysOn>
+        <updateRate>0.0</updateRate>
+        <cameraName>camera1</cameraName>
+        <imageTopicName>image_raw</imageTopicName>
+        <cameraInfoTopicName>camera_info</cameraInfoTopicName>
+        <frameName>camera_link</frameName>
+        <hackBaseline>0.07</hackBaseline>
+        <distortionK1>0.0</distortionK1>
+        <distortionK2>0.0</distortionK2>
+        <distortionK3>0.0</distortionK3>
+        <distortionT1>0.0</distortionT1>
+        <distortionT2>0.0</distortionT2>
+      </plugin>
+    </sensor>
+  </gazebo>
+ <gazebo>
     <plugin name="mpo_700_controller" filename="libgazebo_ros_planar_move.so">
       <commandTopic>cmd_vel</commandTopic>

File: robot_model/mmo_700/urdf/xacros/mpo_700_head.xacro (robot description, xacro)
@@ -1,4 +1,4 @@
 <?xml version="1.0"?>
-<robot xmlns:xacro="http://www.ros.org/wiki/xacro" name="mpo_700">
+<robot xmlns:xacro="http://www.ros.org/wiki/xacro" name="mmo_700">
   <xacro:macro name="mmo_700_head_0" params="name parent *origin">
    <joint name="${name}_joint" type="fixed">
@@ -19,5 +19,5 @@
      <origin xyz="0 0 0.10" rpy="0 0 0"/>
      <geometry>
-        <mesh filename="package://neo_mmo_700/robot_model/mmo_700/meshes/MPO-700-HEAD.dae" scale="0.001 0.001 0.001"/>
+        <mesh filename="package://neo_simulation/robots/mmo_700/meshes/MPO-700-HEAD.dae" scale="0.001 0.001 0.001"/>
      </geometry>
     </visual>
@@ -25,5 +25,5 @@
      <origin xyz="0 0 0.10" rpy="0 0 0" />
      <geometry>
-        <mesh filename="package://neo_mmo_700/robot_model/mmo_700/meshes/MPO-700-HEAD.dae" scale="0.001 0.001 0.001"/>
+        <mesh filename="package://neo_simulation/robots/mmo_700/meshes/MPO-700-HEAD.dae" scale="0.001 0.001 0.001"/>
      </geometry>
     </collision>
@@ -47,5 +47,5 @@
      <origin xyz="0 0 0.10" rpy="0 0 0"/>
      <geometry>
-        <mesh filename="package://neo_mmo_700/robot_model/mmo_700/meshes/MPO-700-HEAD.dae" scale="0.001 0.001 0.001"/>
+        <mesh filename="package://neo_simulation/robots/mmo_700/meshes/MPO-700-HEAD.dae" scale="0.001 0.001 0.001"/>
      </geometry>
     </visual>
@@ -53,5 +53,5 @@
      <origin xyz="0 0 0.10" rpy="0 0 0" />
      <geometry>
-        <mesh filename="package://neo_mmo_700/robot_model/mmo_700/meshes/MPO-700-HEAD.dae" scale="0.001 0.001 0.001"/>
+        <mesh filename="package://neo_simulation/robots/mmo_700/meshes/MPO-700-HEAD.dae" scale="0.001 0.001 0.001"/>
      </geometry>
     </collision>
@@ -75,5 +75,5 @@
      <origin xyz="0 0 0.10" rpy="0 0 0"/>
      <geometry>
-        <mesh filename="package://neo_mmo_700/robot_model/mmo_700/meshes/MPO-700-HEAD.dae" scale="0.001 0.001 0.001"/>
+        <mesh filename="package://neo_simulation/robots/mmo_700/meshes/MPO-700-HEAD.dae" scale="0.001 0.001 0.001"/>
      </geometry>
     </visual>
@@ -81,5 +81,5 @@
      <origin xyz="0 0 0.10" rpy="0 0 0" />
      <geometry>
-        <mesh filename="package://neo_mmo_700/robot_model/mmo_700/meshes/MPO-700-HEAD.dae" scale="0.001 0.001 0.001"/>
+        <mesh filename="package://neo_simulation/robots/mmo_700/meshes/MPO-700-HEAD.dae" scale="0.001 0.001 0.001"/>
      </geometry>
     </collision>
@@ -103,5 +103,5 @@
      <origin xyz="0 0 0.10" rpy="0 0 0"/>
      <geometry>
-        <mesh filename="package://neo_mmo_700/robot_model/mmo_700/meshes/MPO-700-HEAD.dae" scale="0.001 0.001 0.001"/>
+        <mesh filename="package://neo_simulation/robots/mmo_700/meshes/MPO-700-HEAD.dae" scale="0.001 0.001 0.001"/>
      </geometry>
     </visual>
@@ -109,5 +109,5 @@
      <origin xyz="0 0 0.10" rpy="0 0 0" />
      <geometry>
-        <mesh filename="package://neo_mmo_700/robot_model/mmo_700/meshes/MPO-700-HEAD.dae" scale="0.001 0.001 0.001"/>
+        <mesh filename="package://neo_simulation/robots/mmo_700/meshes/MPO-700-HEAD.dae" scale="0.001 0.001 0.001"/>
      </geometry>
     </collision>

File: robot_model/mmo_700/urdf/xacros/mpo_700_wheel.xacro (robot description, xacro)
@@ -1,4 +1,4 @@
 <?xml version="1.0"?>
-<robot xmlns:xacro="http://www.ros.org/wiki/xacro" name="mpo_700">
+<robot xmlns:xacro="http://www.ros.org/wiki/xacro" name="mmo_700">
   <xacro:macro name="mmo_700_wheel" params="name parent *origin">
    <joint name="${name}_joint" type="fixed">

File: robot_model/mmo_700/urdf/xacros/ultrasonic.xacro (robot description, xacro)
@@ -1,4 +1,4 @@
 <?xml version="1.0"?>
-<robot xmlns:xacro="http://www.ros.org/wiki/xacro" name="mp_400">
+<robot xmlns:xacro="http://www.ros.org/wiki/xacro" name="mmo_700">
   <xacro:macro name="us_sensor" params="name parent *origin">
     <joint name="${name}_joint" type="fixed">

Commit message: sensors added on the corner

File: robot_model/mmo_700/mmo_700.urdf.xacro (robot description, xacro)
@@ -52,8 +52,10 @@
 <!-- Sensors -->
   <xacro:sick_laser_v0 name="lidar_1" parent="base_link" ros_topic="lidar_1/scan_filtered">
-    <origin xyz="0.360 0 0.181" rpy="3.14 0 0 " />
+  <!--<origin xyz="0.360 0 0.181" rpy="3.14 0 0" />-->
+    <origin xyz="0.338 0.288 0.223" rpy="3.14 0 0.79" /> <!-- Scanners on the side -->
   </xacro:sick_laser_v0>
   <xacro:sick_laser_v0 name="lidar_2" parent="base_link" ros_topic="lidar_2/scan_filtered">
-    <origin xyz="-0.360 0 0.181" rpy="3.14 0 3.14" />
+  <!--<origin xyz="-0.360 0 0.181" rpy="3.14 0 3.14" />-->
+    <origin xyz="-0.338 -0.288 0.223" rpy="3.14 0 3.93" /> <!-- Scanners on the side -->
   </xacro:sick_laser_v0>
      <!--+++++++++++++++++++ IMU ++++++++++++++++++++++++-->
